File: Test-Stand/Test.kicad_pcb (KiCad board)
At the start: 2 copper layers, 78.2 x 61 mm, 21 parts, among them J1 Conn_01x04_Pin, J2 Conn_01x03_Pin, J3 XT90PW-F, J4 XT90PW-F, Q1 S8550 2TY DNP SOT-23 SMD 0.5A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, U1 LM741, U3 HX711, U4 MPXV7002DP

Commit message: Updated project files
Parts:
- removed J2: Conn_01x03_Pin, Connector_JST:JST_EH_B3B-EH-A_1x03_P2.50mm_Vertical
- moved J3 28.1 mm to (102.3, 96.5)
- moved R2 12.0 mm to (107.2, 110.8)
- moved R3 12.0 mm to (111.2, 110.8)
- moved C5 11.2 mm to (109.2, 121.7)
- moved J4 9.25 mm to (114.3, 96.5), turned to 0 degrees
- moved U2 5.96 mm to (105.0, 100.1), turned to 0 degrees
Connections:
- A1 pad 17: Net-(A1-3V3) -> unconnected-(A1-3V3-Pad17)
- A1 pad 6: Net-(A1-D3) -> unconnected-(A1-D3-Pad6)
- U4 pad 2: Net-(A1-3V3) -> Net-(A1-+5V)
Routing:
- net Net-(A1-+5V): track 64.0 -> 95.8 mm, vias 2 -> 3
- net Net-(U1-+): track 60.7 -> 40.3 mm
- net Net-(A1-3V3): track 19.0 -> 0.00 mm
- net GND: track 198.4 -> 216.9 mm
- net Net-(A1-D3): track 11.2 -> 0.00 mm
- net Net-(J4-Pos): track 23.4 -> 13.6 mm
- net Net-(J3-Pos): track 8.84 -> 0.00 mm
- net Net-(A1-A7): track 28.5 -> 29.4 mm
Other:
- board size 78.2 x 61 mm -> 75.7 x 61 mm

Commit message: Updated test stand files
Parts:
- added J2: Conn_01x06, Connector_JST:JST_EH_B6B-EH-A_1x06_P2.50mm_Vertical, F.Cu at (134.6, 76.2)
Connections:
- A1 pad 17: unconnected-(A1-3V3-Pad17) -> Net-(A1-3V3)
- A1 pad 5: unconnected-(A1-D2-Pad5) -> Net-(A1-D2)
- A1 pad 6: unconnected-(A1-D3-Pad6) -> Net-(A1-D3)
- A1 pad 7: unconnected-(A1-D4-Pad7) -> Net-(A1-D4)
- A1 pad 8: unconnected-(A1-D5-Pad8) -> Net-(A1-D5)
- U2 pad 1: Net-(A1-+5V) -> Net-(A1-3V3)
Routing:
- net Net-(A1-3V3): track 0.00 -> 61.1 mm
- net Net-(A1-D5): track 0.00 -> 31.7 mm
- net Net-(A1-D4): track 0.00 -> 28.1 mm
- net Net-(A1-D3): track 0.00 -> 24.6 mm
- net Net-(A1-D2): track 0.00 -> 21.0 mm
- net Net-(A1-+5V): track 95.8 -> 81.0 mm, vias 3 -> 4
- added copper zone on B.Cu, net GND
