File: Test-Stand/Test.kicad_sch (KiCad schematic)
At the start: 21 parts, among them J1 Conn_01x04_Pin, J2 Conn_01x03_Pin, J3 XT90PW-F, J4 XT90PW-F, Q1 S8550 2TY DNP SOT-23 SMD 0.5A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, U1 LM741, U3 HX711, U4 MPXV7002DP

Commit message: Updated project files
Parts:
- removed J2: Conn_01x03_Pin, Connector_JST:JST_EH_B3B-EH-A_1x03_P2.50mm_Vertical, symbol Connector:Screw_Terminal_01x03
Connections:
- net GND: now also U2.4 (NC), U2.7 (NC)
- net at A1.27 (+5V), C6.1, Q1.3 (E)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: now also U4.2 (VS)
- net at A1.17 (3V3): no longer U4.2 (VS)
- no-connect marks 0 -> 27
Changed lines of the file:
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@@
   (junction (at 123.19 35.56) (diameter 0) (color 0 0 0 0)
   )
-  (junction (at 146.05 173.99) (diameter 0) (color 0 0 0 0)
-  )
-  (junction (at 208.28 105.41) (diameter 0) (color 0 0 0 0)
-  )
   (junction (at 142.24 149.86) (diameter 0) (color 0 0 0 0)
   )
@@
   (junction (at 107.95 173.99) (diameter 0) (color 0 0 0 0)
   )
+  (junction (at 176.53 125.73) (diameter 0) (color 0 0 0 0)
+  )
   (junction (at 86.36 173.99) (diameter 0) (color 0 0 0 0)
   )
@@
   (junction (at 170.18 43.18) (diameter 0) (color 0 0 0 0)
   )
+  (junction (at 176.53 135.89) (diameter 0) (color 0 0 0 0)
+  )
   (junction (at 90.17 147.32) (diameter 0) (color 0 0 0 0)
   )
@@
   (junction (at 107.95 147.32) (diameter 0) (color 0 0 0 0)
   )
-  (wire (pts (xy 63.5 102.87) (xy 146.05 102.87))
-    (stroke (width 0) (type default))
-  )
+  (no_connect (at 240.03 130.81))
+  (no_connect (at 214.63 105.41))
+  (no_connect (at 214.63 128.27))
+  (no_connect (at 240.03 128.27))
+  (no_connect (at 214.63 138.43))
+  (no_connect (at 214.63 107.95))
+  (no_connect (at 240.03 107.95))
+  (no_connect (at 214.63 130.81))
+  (no_connect (at 134.62 149.86))
+  (no_connect (at 214.63 123.19))
+  (no_connect (at 214.63 110.49))
+  (no_connect (at 224.79 95.25))
+  (no_connect (at 214.63 133.35))
+  (no_connect (at 214.63 120.65))
+  (no_connect (at 127 142.24))
+  (no_connect (at 214.63 118.11))
+  (no_connect (at 214.63 135.89))
+  (no_connect (at 240.03 115.57))
+  (no_connect (at 132.08 157.48))
+  (no_connect (at 181.61 35.56))
+  (no_connect (at 129.54 157.48))
+  (no_connect (at 214.63 113.03))
+  (no_connect (at 240.03 105.41))
+  (no_connect (at 127 157.48))
+  (no_connect (at 214.63 115.57))
+  (no_connect (at 214.63 125.73))
+  (no_connect (at 240.03 133.35))
   (wire (pts (xy 212.09 38.1) (xy 213.36 38.1))
     (stroke (width 0) (type default))
@@
     (stroke (width 0) (type default))
   )
-  (wire (pts (xy 251.46 91.44) (xy 229.87 91.44))
-    (stroke (width 0) (type default))
-  )
   (wire (pts (xy 214.63 80.01) (xy 123.19 80.01))
     (stroke (width 0) (type default))
   )
-  (wire (pts (xy 208.28 105.41) (xy 208.28 129.54))
+  (wire (pts (xy 208.28 86.36) (xy 208.28 129.54))
     (stroke (width 0) (type default))
   )
@@
     (stroke (width 0) (type default))
   )
+  (wire (pts (xy 176.53 118.11) (xy 176.53 125.73))
+    (stroke (width 0) (type default))
+  )
   (wire (pts (xy 72.39 137.16) (xy 82.55 137.16))
     (stroke (width 0) (type default))
@@
     (stroke (width 0) (type default))
   )
-  (wire (pts (xy 251.46 119.38) (xy 251.46 91.44))
-    (stroke (width 0) (type default))
-  )
-  (wire (pts (xy 176.53 125.73) (xy 176.53 173.99))
+  (wire (pts (xy 163.83 118.11) (xy 176.53 118.11))
+    (stroke (width 0) (type default))
+  )
+  (wire (pts (xy 251.46 86.36) (xy 251.46 119.38))
+    (stroke (width 0) (type default))
+  )
+  (wire (pts (xy 176.53 125.73) (xy 176.53 135.89))
     (stroke (width 0) (type default))
   )
@@
     (stroke (width 0) (type default))
   )
+  (wire (pts (xy 251.46 86.36) (xy 232.41 86.36))
+    (stroke (width 0) (type default))
+  )
   (wire (pts (xy 207.01 151.13) (xy 251.46 151.13))
     (stroke (width 0) (type default))
@@
     (stroke (width 0) (type default))
   )
+  (wire (pts (xy 163.83 135.89) (xy 176.53 135.89))
+    (stroke (width 0) (type default))
+  )
   (wire (pts (xy 179.07 173.99) (xy 227.33 173.99))
     (stroke (width 0) (type default))
@@
     (stroke (width 0) (type default))
   )
-  (wire (pts (xy 229.87 91.44) (xy 229.87 95.25))
-    (stroke (width 0) (type default))
-  )
-  (wire (pts (xy 107.95 173.99) (xy 146.05 173.99))
-    (stroke (width 0) (type default))
-  )
   (wire (pts (xy 243.84 52.07) (xy 243.84 120.65))
     (stroke (width 0) (type default))
@@
     (stroke (width 0) (type default))
   )
-  (wire (pts (xy 205.74 107.95) (xy 205.74 113.03))
-    (stroke (width 0) (type default))
-  )
-  (wire (pts (xy 146.05 173.99) (xy 176.53 173.99))
+  (wire (pts (xy 107.95 173.99) (xy 176.53 173.99))
     (stroke (width 0) (type default))
   )
@@
     (stroke (width 0) (type default))
   )
-  (wire (pts (xy 205.74 113.03) (xy 214.63 113.03))
-    (stroke (width 0) (type default))
-  )
-  (wire (pts (xy 63.5 105.41) (xy 208.28 105.41))
-    (stroke (width 0) (type default))
-  )
   (wire (pts (xy 172.72 125.73) (xy 176.53 125.73))
     (stroke (width 0) (type default))
@@
     (stroke (width 0) (type default))
   )
+  (wire (pts (xy 176.53 135.89) (xy 176.53 173.99))
+    (stroke (width 0) (type default))
+  )
   (wire (pts (xy 201.93 69.85) (xy 201.93 68.58))
     (stroke (width 0) (type default))
@@
     (stroke (width 0) (type default))
   )
-  (wire (pts (xy 146.05 102.87) (xy 146.05 173.99))
-    (stroke (width 0) (type default))
-  )
   (wire (pts (xy 198.12 68.58) (xy 179.07 68.58))
     (stroke (width 0) (type default))
@@
     (stroke (width 0) (type default))
   )
-  (wire (pts (xy 208.28 86.36) (xy 208.28 105.41))
-    (stroke (width 0) (type default))
-  )
   (wire (pts (xy 232.41 86.36) (xy 232.41 38.1))
     (stroke (width 0) (type default))
@@
     (stroke (width 0) (type default))
   )
+  (wire (pts (xy 163.83 133.35) (xy 163.83 135.89))
+    (stroke (width 0) (type default))
+  )
   (wire (pts (xy 246.38 123.19) (xy 246.38 54.61))
     (stroke (width 0) (type default))
@@
   )
   (wire (pts (xy 213.36 38.1) (xy 213.36 27.94))
-    (stroke (width 0) (type default))
-  )
-  (wire (pts (xy 63.5 107.95) (xy 205.74 107.95))
     (stroke (width 0) (type default))
   )
@@
   (text "ESC" (at 58.42 132.08 0)
     (effects (font (size 1.27 1.27)) (justify left bottom))
-  )
-  (symbol (lib_id "Connector:Screw_Terminal_01x03") (at 58.42 105.41 180) (unit 1)
-    (in_bom yes) (on_board yes) (dnp no) (fields_autoplaced)
-    (property "Reference" "J2" (at 58.42 96.52 0)
-      (effects (font (size 1.27 1.27)))
-    )
-    (property "Value" "Conn_01x03_Pin" (at 58.42 99.06 0)
-      (effects (font (size 1.27 1.27)))
-    )
-    (property "Footprint" "Connector_JST:JST_EH_B3B-EH-A_1x03_P2.50mm_Vertical" (at 58.42 105.41 0)
-      (effects (font (size 1.27 1.27)) hide)
-    )
-    (property "Datasheet" "~" (at 58.42 105.41 0)
-      (effects (font (size 1.27 1.27)) hide)
-    )
-    (pin "1")
-    (pin "2")
-    (pin "3")
-    (instances
-      (project "Test"
-        (path "/5de3e6fd-b8e3-4ef4-89d0-61c729b79836"
-          (reference "J2") (unit 1)
-        )
-      )
-    )
   )
   (symbol (lib_id "Device:R_US") (at 91.44 86.36 90) (unit 1)
@@
       (effects (font (size 1.27 1.27)) hide)
     )
+    (pin "1")
+    (pin "2")
+    (pin "3")
+    (pin "4")
     (pin "5")
     (pin "6")
     (pin "7")
-    (pin "4")
-    (pin "2")
-    (pin "1")
-    (pin "3")
-    (instances
-      (project "Test"
+    (instances
+      (project "Test"

Commit message: Updated test stand files
Parts:
- added J2: Conn_01x06, Connector_JST:JST_EH_B6B-EH-A_1x06_P2.50mm_Vertical, symbol Connector_Generic:Conn_01x06
Connections:
- net GND: now also J2.6 (Pin_6)
- net at A1.27 (+5V), C6.1, Q1.3 (E)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: now also J2.5 (Pin_5); no longer U2.1 (vcc)
- net at A1.17 (3V3): now also U2.1 (vcc)
- net at A1.5 (D2): now also J2.4 (Pin_4)
- net at A1.6 (D3): now also J2.3 (Pin_3)
- net at A1.7 (D4): now also J2.2 (Pin_2)
- net at A1.8 (D5): now also J2.1 (Pin_1)
- no-connect marks 27 -> 23
Other:
- note added: "Checked"
- note added: "Checked 1x4"
- note added: "Checked C1"
- note added: "Checked C3"
- note added: "Checked C4"
- note added: "Checked C6"
- note added: "Checked R1"
- note added: "Checked R4"
- note added: "Checked R5"
- note added: "Checked R6"
- note added: "Checked Transistor"
- note added: "Checked buffer"
- note added: "Checked magnometer"
- note added: "Micro SD Module"
Changed lines of the file:
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@@
   (junction (at 227.33 173.99) (diameter 0) (color 0 0 0 0)
+  )
+  (junction (at 176.53 118.11) (diameter 0) (color 0 0 0 0)
   )
   (junction (at 232.41 86.36) (diameter 0) (color 0 0 0 0)
@@
   (no_connect (at 134.62 149.86))
   (no_connect (at 214.63 123.19))
-  (no_connect (at 214.63 110.49))
   (no_connect (at 224.79 95.25))
   (no_connect (at 214.63 133.35))
   (no_connect (at 214.63 120.65))
   (no_connect (at 127 142.24))
-  (no_connect (at 214.63 118.11))
   (no_connect (at 214.63 135.89))
   (no_connect (at 240.03 115.57))
@@
   (no_connect (at 181.61 35.56))
   (no_connect (at 129.54 157.48))
-  (no_connect (at 214.63 113.03))
   (no_connect (at 240.03 105.41))
   (no_connect (at 127 157.48))
-  (no_connect (at 214.63 115.57))
   (no_connect (at 214.63 125.73))
   (no_connect (at 240.03 133.35))
+  (wire (pts (xy 205.74 118.11) (xy 214.63 118.11))
+    (stroke (width 0) (type default))
+  )
+  (wire (pts (xy 210.82 100.33) (xy 210.82 110.49))
+    (stroke (width 0) (type default))
+  )
   (wire (pts (xy 212.09 38.1) (xy 213.36 38.1))
     (stroke (width 0) (type default))
@@
     (stroke (width 0) (type default))
   )
+  (wire (pts (xy 229.87 92.71) (xy 193.04 92.71))
+    (stroke (width 0) (type default))
+  )
   (wire (pts (xy 106.68 67.31) (xy 80.01 67.31))
     (stroke (width 0) (type default))
@@
     (stroke (width 0) (type default))
   )
-  (wire (pts (xy 208.28 86.36) (xy 208.28 129.54))
-    (stroke (width 0) (type default))
-  )
   (wire (pts (xy 107.95 160.02) (xy 107.95 173.99))
     (stroke (width 0) (type default))
@@
     (stroke (width 0) (type default))
   )
+  (wire (pts (xy 210.82 110.49) (xy 214.63 110.49))
+    (stroke (width 0) (type default))
+  )
   (wire (pts (xy 254 135.89) (xy 240.03 135.89))
     (stroke (width 0) (type default))
   )
-  (wire (pts (xy 172.72 129.54) (xy 208.28 129.54))
-    (stroke (width 0) (type default))
-  )
   (wire (pts (xy 72.39 160.02) (xy 82.55 160.02))
     (stroke (width 0) (type default))
@@
     (stroke (width 0) (type default))
   )
+  (wire (pts (xy 208.28 113.03) (xy 214.63 113.03))
+    (stroke (width 0) (type default))
+  )
   (wire (pts (xy 107.95 173.99) (xy 90.17 173.99))
     (stroke (width 0) (type default))
@@
     (stroke (width 0) (type default))
   )
+  (wire (pts (xy 205.74 107.95) (xy 205.74 118.11))
+    (stroke (width 0) (type default))
+  )
+  (wire (pts (xy 207.01 105.41) (xy 207.01 115.57))
+    (stroke (width 0) (type default))
+  )
   (wire (pts (xy 72.39 67.31) (xy 57.15 67.31))
     (stroke (width 0) (type default))
@@
     (stroke (width 0) (type default))
   )
+  (wire (pts (xy 193.04 92.71) (xy 193.04 129.54))
+    (stroke (width 0) (type default))
+  )
   (wire (pts (xy 227.33 52.07) (xy 243.84 52.07))
     (stroke (width 0) (type default))
@@
     (stroke (width 0) (type default))
   )
+  (wire (pts (xy 157.48 100.33) (xy 210.82 100.33))
+    (stroke (width 0) (type default))
+  )
   (wire (pts (xy 163.83 135.89) (xy 176.53 135.89))
     (stroke (width 0) (type default))
@@
     (stroke (width 0) (type default))
   )
+  (wire (pts (xy 157.48 95.25) (xy 176.53 95.25))
+    (stroke (width 0) (type default))
+  )
   (wire (pts (xy 261.62 124.46) (xy 248.92 124.46))
     (stroke (width 0) (type default))
@@
     (stroke (width 0) (type default))
   )
+  (wire (pts (xy 157.48 107.95) (xy 205.74 107.95))
+    (stroke (width 0) (type default))
+  )
   (wire (pts (xy 142.24 149.86) (xy 137.16 149.86))
     (stroke (width 0) (type default))
@@
     (stroke (width 0) (type default))
   )
+  (wire (pts (xy 157.48 102.87) (xy 208.28 102.87))
+    (stroke (width 0) (type default))
+  )
   (wire (pts (xy 123.19 64.77) (xy 107.95 64.77))
     (stroke (width 0) (type default))
@@
     (stroke (width 0) (type default))
   )
+  (wire (pts (xy 176.53 95.25) (xy 176.53 118.11))
+    (stroke (width 0) (type default))
+  )
   (wire (pts (xy 135.89 43.18) (xy 135.89 35.56))
     (stroke (width 0) (type default))
@@
     (stroke (width 0) (type default))
   )
+  (wire (pts (xy 157.48 97.79) (xy 210.82 97.79))
+    (stroke (width 0) (type default))
+  )
+  (wire (pts (xy 229.87 95.25) (xy 229.87 92.71))
+    (stroke (width 0) (type default))
+  )
   (wire (pts (xy 172.72 125.73) (xy 176.53 125.73))
     (stroke (width 0) (type default))
@@
     (stroke (width 0) (type default))
   )
+  (wire (pts (xy 193.04 129.54) (xy 172.72 129.54))
+    (stroke (width 0) (type default))
+  )
   (wire (pts (xy 121.92 147.32) (xy 107.95 147.32))
     (stroke (width 0) (type default))
@@
     (stroke (width 0) (type default))
   )
+  (wire (pts (xy 210.82 97.79) (xy 210.82 86.36))
+    (stroke (width 0) (type default))
+  )
   (wire (pts (xy 248.92 125.73) (xy 240.03 125.73))
     (stroke (width 0) (type default))
@@
     (stroke (width 0) (type default))
   )
+  (wire (pts (xy 207.01 115.57) (xy 214.63 115.57))
+    (stroke (width 0) (type default))
+  )
   (wire (pts (xy 198.12 68.58) (xy 179.07 68.58))
     (stroke (width 0) (type default))
@@
     (stroke (width 0) (type default))
   )
+  (wire (pts (xy 210.82 86.36) (xy 232.41 86.36))
+    (stroke (width 0) (type default))
+  )
   (wire (pts (xy 83.82 41.91) (xy 96.52 41.91))
     (stroke (width 0) (type default))
@@
     (stroke (width 0) (type default))
   )
-  (wire (pts (xy 208.28 86.36) (xy 232.41 86.36))
+  (wire (pts (xy 157.48 105.41) (xy 207.01 105.41))
     (stroke (width 0) (type default))
   )
@@
     (stroke (width 0) (type default))
   )
+  (wire (pts (xy 208.28 102.87) (xy 208.28 113.03))
+    (stroke (width 0) (type default))
+  )
+  (text "Checked R4" (at 86.36 91.44 0)
+    (effects (font (size 1.27 1.27)) (justify left bottom))
+  )
+  (text "Checked R6" (at 125.73 57.15 0)
+    (effects (font (size 1.27 1.27)) (justify left bottom))
+  )
+  (text "Checked Transistor" (at 152.4 33.02 0)
+    (effects (font (size 1.27 1.27)) (justify left bottom))
+  )
+  (text "Checked R1" (at 71.12 71.12 0)
+    (effects (font (size 1.27 1.27)) (justify left bottom))
+  )
+  (text "Checked C3" (at 83.82 60.96 0)
+    (effects (font (size 1.27 1.27)) (justify left bottom))
+  )
+  (text "Checked C1" (at 82.55 38.1 0)
+    (effects (font (size 1.27 1.27)) (justify left bottom))
+  )
   (text "Battery" (at 59.69 158.75 0)
     (effects (font (size 1.27 1.27)) (justify left bottom))
   )
   (text "ESC" (at 58.42 132.08 0)
+    (effects (font (size 1.27 1.27)) (justify left bottom))
+  )
+  (text "Checked R5" (at 109.22 40.64 0)
+    (effects (font (size 1.27 1.27)) (justify left bottom))
+  )
+  (text "Micro SD Module" (at 129.54 95.25 0)
+    (effects (font (size 1.27 1.27)) (justify left bottom))
+  )
+  (text "Checked\n" (at 275.59 109.22 0)
+    (effects (font (size 1.27 1.27)) (justify left bottom))
+  )
+  (text "Checked 1x4\n" (at 21.59 24.13 0)
+    (effects (font (size 1.27 1.27)) (justify left bottom))
+  )
+  (text "Checked magnometer" (at 152.4 116.84 0)
+    (effects (font (size 1.27 1.27)) (justify left bottom))
+  )
+  (text "Checked C4" (at 114.3 83.82 0)
+    (effects (font (size 1.27 1.27)) (justify left bottom))
+  )
+  (text "Checked buffer" (at 129.54 140.97 0)
+    (effects (font (size 1.27 1.27)) (justify left bottom))
+  )
+  (text "Checked C6" (at 154.94 22.86 0)
     (effects (font (size 1.27 1.27)) (justify left bottom))
   )
@@
         )
       )
+    )
+  )
+  (symbol (lib_id "Connector_Generic:Conn_01x06") (at 152.4 102.87 180) (unit 1)
+    (in_bom yes) (on_board yes) (dnp no) (fields_autoplaced)
+    (property "Reference" "J2" (at 152.4 88.9 0)
+      (effects (font (size 1.27 1.27)))
+    )
+    (property "Value" "Conn_01x06" (at 152.4 91.44 0)
+      (effects (font (size 1.27 1.27)))
+    )
+    (property "Footprint" "Connector_JST:JST_EH_B6B-EH-A_1x06_P2.50mm_Vertical" (at 152.4 102.87 0)
+      (effects (font (size 1.27 1.27)) hide)
+    )
+    (property "Datasheet" "~" (at 152.4 102.87 0)
+      (effects (font (size 1.27 1.27)) hide)
+    )
+    (pin "1")
+    (pin "2")
+    (pin "3")
+    (pin "4")
+    (pin "5")
+    (pin "6")
+    (instances
+      (project "Test"
+        (path "/5de3e6fd-b8e3-4ef4-89d0-61c729b79836"
+          (reference "J2") (unit 1)
+        )
+      )
